Commit message: Changed color name of black to sawyer_black, this will prevent conflicts with generic color names when the sawyer urdf is combined with another urdf

File: sawyer_description/urdf/sawyer_base.urdf.xacro (robot description, xacro)
@@ -3,5 +3,5 @@
   <xacro:arg name="gazebo" default="false"/>
   <xacro:arg name="pedestal" default="true"/>
-  <material name="black">
+  <material name="sawyer_black">
     <color rgba="0 0 0 1"/>
   </material>
